Commit message: change base_mobile_link name to base_link

File: agvbot_description/urdf/mech/base_link.xacro (robot description, xacro)
@@ -10,5 +10,5 @@
     <xacro:property name="imu_height" value="0.002" />
     <xacro:property name="lidar_radius" value="0.025" />
-    <xacro:property name="lidar_length" value="0.05" />
+    <xacro:property name="lidar_length" value="0.03" />
     <link name="base_footprint"/>
     <link name="base_link">
@@ -29,5 +29,5 @@
                            o_xyz="0 0 ${base_height / 2.0}" o_rpy="0 0 0" />
     </link>
-    <joint name="base_joint" type="fixed">
+    <joint name="base_moblile_joint" type="fixed">
         <parent link="base_footprint" />
         <child link="base_link" />
