Commit message: adding depth camera

File: agvbot_description/urdf/sensors/lidar_link.xacro (robot description, xacro)
@@ -21,5 +21,5 @@
         <parent link="base_link" />
         <child link="lidar_link" />
-        <origin xyz="${(base_length/2.0)-lidar_radius} 0 ${base_height + lidar_length}" rpy="0 0 0"/>
+        <origin xyz="${base_length/2-lidar_radius} 0 ${base_height+lidar_length/2}" rpy="0 0 0"/>
     </joint>
 </robot>
